Commit message: add custom geometries; set explicit joint/dof values

File: model.urdf (robot description, URDF)
Before this commit: robot dummy3r, 5 links, 4 joints
Joints:
- joint joint0: origin rpy=0 0 1.5708 -> (none)
- joint joint1: axis (none) -> 0 1 0
- joint joint2: axis (none) -> 0 1 0
- joint joint3: axis (none) -> 0 1 0

Commit message: fix link4 length to 0.1

File: model.urdf (robot description, URDF)
Before this commit: robot dummy3r, 5 links, 4 joints
Links:
- link link4: geometry visual cylinder length=.08 radius=.04; visual cylinder length=.1 radius=.03
